File: BUTTeRUSEr_PTM.sch (KiCad schematic (older format))
At the start: 2 parts, among them P1 BATT, P2 OUT

Commit message: Update schematics
Parts:
- removed P1: BATT, symbol CONN_01X02
- removed P2: OUT, symbol CONN_01X02
- added C1: 4.7uF, Capacitors_SMD:C_0805_HandSoldering, symbol C
- added C2: 33pF, Capacitors_SMD:C_0805_HandSoldering, symbol C
- added C3, C4: 22uF, Capacitors_SMD:C_0805_HandSoldering, symbol C
- added C5: 2.2uF, Capacitors_SMD:C_0805_HandSoldering, symbol C
- added C6: 10uF, Capacitors_SMD:C_0805_HandSoldering, symbol C
- added C7: 0.1uF, Capacitors_SMD:C_0805_HandSoldering, symbol C
- added C8: 68uF, Capacitors_SMD:C_0805_HandSoldering, symbol C
- added C9: 1uF, Capacitors_SMD:C_0805_HandSoldering, symbol C
- added D1: MBRA140, Diodes_SMD:DO-214AB_Handsoldering, symbol D
- added D2, D3: KPTR-3216EC, LEDs:LED-1206, symbol LED
- added JP1, JP2: Jumper_NO_Small, Resistors_SMD:R_0603, symbol Jumper_NO_Small
- added L1: 2.2uH, MonkeyLive:ELL6SH047M, symbol L_Small
- added L2: 47uH, MonkeyLive:SRR0604-2R2ML, symbol L_Small
- added P1: B+, Socket_Strips:Socket_Strip_Straight_1x01, symbol CONN_01X01
- added P2: B-, Socket_Strips:Socket_Strip_Straight_1x01, symbol CONN_01X01
- added P3: O+, Socket_Strips:Socket_Strip_Straight_1x01, symbol CONN_01X01
- added P4: O-, Socket_Strips:Socket_Strip_Straight_1x01, symbol CONN_01X01
- added Q1, Q2: BC850, Housings_SOT-23_SOT-143_TSOT-6:SOT-23_Handsoldering, symbol BC850
- added R1, R3: 499K, Resistors_SMD:R_0805_HandSoldering, symbol R
- added R2: 124K, Resistors_SMD:R_0805_HandSoldering, symbol R
- added R4: 1K, Resistors_SMD:R_0805_HandSoldering, symbol R
- added R5: 470K, Resistors_SMD:R_0805_HandSoldering, symbol R
- added R6, R7: 330, Resistors_SMD:R_0805_HandSoldering, symbol R
- added U1: LTC3539EDCB, MonkeyLive:LTC3539, symbol LTC3539EDCB
- added U2: NCP1402 33T1, Housings_SOT-23_SOT-143_TSOT-6:SOT-23-5, symbol NCP1402
- added U3: LMC555, Housings_SOIC:SOIC-8_3.9x4.9mm_Pitch1.27mm, symbol LM555N
Connections:
- net labels added: +3.3V
- wire segments 6 -> 95
- no-connect marks 0 -> 2
Other:
- note added: "Common part"
- note added: "Crazy Option"
- note added: "LITE EDITION \nNO LONGUER\nSUPPORTED"
- note added: "Lite Edition"
- note added: "Pro Edition"
- note removed: "BUTTeRUSEr rev 5.3\n\nProbe The Monkey Edition"
